File: electrical/OutdoorWarningLight.sch (KiCad schematic (older format))
At the start: 22 parts

Commit message: Add firmware
Parts:
- removed C? (x2): 1uF, symbol device:C
- removed Q?: BF245B, Package_TO_SOT_THT:TO-92_Inline, symbol Transistor_FET:BF245B
- added C1, C2: 1uF, symbol device:CP
- added Q1: BS170, Package_TO_SOT_THT:TO-92_Inline, symbol Transistor_FET:BS170
- added R1: 100k, symbol device:R
- added R2: 1k, symbol device:R
- gave numbers to parts that had none: 19
Connections:
- net +3V3: now also C2.1, R1.1
- net GND: now also C1.2, C2.2, Q1.3 (S)
- net at Q2.1 (D), U2.3 (VI): now also C1.1
- net at Q2.2 (G), R4.2, SW1.2: now also Q1.1 (D)
- net at U1.2 (XTAL1/PB3): now also R2.2
- new net: Q1.2 (G), R1.2, R2.1
Other:
- moved on the sheet: J1, Q2, R4, SW1, U2

Commit message: Add PCB layout
Parts:
- removed Q1: BS170, Package_TO_SOT_THT:TO-92_Inline, symbol Transistor_FET:BS170
- removed Q3, Q4, Q5, Q6: BD135, Package_TO_SOT_THT:TO-126-3_Vertical, symbol Transistor_BJT:BD135
- removed SW1: SW_Push, symbol switches:SW_Push
- added C3: 0.1uF, Capacitor_SMD:C_0603_1608Metric, symbol Device:C
- added J6: SW, Connector_PinSocket_2.54mm:PinSocket_1x02_P2.54mm_Horizontal, symbol Connector_Generic:Conn_01x02
- added J7: AVR-ISP-6, Connector_PinHeader_2.54mm:PinHeader_2x03_P2.54mm_Vertical, symbol Connector:AVR-ISP-6
- added Q1, Q3, Q4, Q5, Q6: BSS214, Package_TO_SOT_SMD:SOT-23, symbol Device:Q_NMOS_GSD
- C1, C2: footprint (none) -> Capacitor_THT:CP_Radial_D5.0mm_P2.00mm; symbol device:CP -> OutdoorWarningLight-rescue:CP-device
- J1: value LED1 -> BAT; footprint (none) -> Connector_PinSocket_2.54mm:PinSocket_1x02_P2.54mm_Horizontal
- J2, J3, J4, J5: footprint (none) -> Connector_PinSocket_2.54mm:PinSocket_1x02_P2.54mm_Horizontal
- Q2: footprint Package_TO_SOT_THT:TO-92_Inline -> Package_TO_SOT_SMD:SOT-23
- R1, R2, R3: footprint (none) -> Resistor_SMD:R_0603_1608Metric; symbol device:R -> OutdoorWarningLight-rescue:R-device
- R4, R5, R6, R7, R8: footprint (none) -> Resistor_SMD:R_0603_1608Metric; symbol device:R_Small -> OutdoorWarningLight-rescue:R_Small-device
- U1: value ATtiny85-20PU -> ATtiny85-SO; footprint Package_DIP:DIP-8_W7.62mm -> Package_SO:SOIC-8_3.9x4.9mm_P1.27mm; symbol MCU_Microchip_ATtiny:ATtiny85-20PU -> OutdoorWarningLight-rescue:ATtiny85-20PU-MCU_Microchip_ATtiny
Connections:
- net +3V3: now also C3.1, J7.2 (VCC)
- net GND: now also C3.2, J6.1 (Pin_1), J7.6 (GND), Q1.2 (S), Q3.2 (S), Q4.2 (S), Q5.2 (S), Q6.2 (S)
- net at Q2.2 (G), R4.2: now also J6.2 (Pin_2), Q1.3 (D)
- net at R3.2, U1.1 (~RESET~/PB5): now also J7.5 (~RST)
- net at R5.2, U1.5 (AREF/PB0): now also J7.4 (MOSI)
- net at R6.2, U1.6 (PB1): now also J7.1 (MISO)
- net at R7.2, U1.7 (PB2): now also J7.3 (SCK)
- net at R1.2, R2.1: now also Q1.1 (G)
- net at J2.2 (Pin_2): now also Q3.3 (D)
- net at R5.1: now also Q3.1 (G)
- net at J3.2 (Pin_2): now also Q4.3 (D)
- net at R6.1: now also Q4.1 (G)
- net at J4.2 (Pin_2): now also Q5.3 (D)
- net at R7.1: now also Q5.1 (G)
- net at J5.2 (Pin_2): now also Q6.3 (D)
- net at R8.1: now also Q6.1 (G)
Other:
- moved on the sheet: U1
